File: PCB/Tesla Coil MIDI Synth.kicad_pcb (KiCad board)
At the start: 4 copper layers, 132.1 x 61 mm, 102 parts, among them J1 USB C, J2 JTAG, J3 Expansion, J4 Headphone Output, J5 BNC Output, J6 MIDI Out, J7 MIDI In, Q1 2N7002, Q2 2N7002, SW1 Reset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

Commit message: fixed PCB
 * Added 5.1k resistors to CC lines on USB-C port
 * Replaced diode OR thing and MOSFET with too low of a threshold voltage with a real OR gate and buffer
 * Fixed polarity of BNC output
 * Made headphone output not murderously loud and asymmetric
 * Added direct in/out to expansion pins
 * Reduced impedance into ADC for average volume level sensing
 * Increased MIDI input pullup resistance
 * Made thermal spokes to copper planes thinner
Parts:
- removed D10, D11, D12, D13, D14, D9: D, Diode_SMD:D_SOD-123
- removed Q1, Q2: 2N7002, Package_TO_SOT_SMD:SOT-23
- removed the REF** at (28.2, 42.7)
- added C26: 100n, Capacitor_SMD:C_0603_1608Metric_Pad1.08x0.95mm_HandSolder, F.Cu at (124.6, 46.5)
- added R28: 5.1k, Resistor_SMD:R_0603_1608Metric_Pad0.98x0.95mm_HandSolder, F.Cu at (25.5, 30.5)
- added U8: 4075, Package_SO:SOIC-14_3.9x8.7mm_P1.27mm, F.Cu at (122.2, 52.2)
- added U9: 74LVC1G17, Package_TO_SOT_SMD:SOT-23-5, F.Cu at (127.8, 49.5)
- C24: value 100n -> 10µ; footprint Capacitor_SMD:C_0603_1608Metric_Pad1.08x0.95mm_HandSolder -> Capacitor_SMD:C_0805_2012Metric_Pad1.18x1.45mm_HandSolder
- J3: footprint Connector_PinHeader_2.54mm:PinHeader_2x05_P2.54mm_Vertical -> Connector_PinHeader_2.54mm:PinHeader_2x06_P2.54mm_Vertical
- R16: value 1k -> 5.1k
- R17: value 2.2k -> 10k
- R18, R19: value 47 -> 100
- R21: value 47 -> 220
- R22: value 47 -> 10k
- R27: value 100k -> 10k
- moved R16 97.4 mm to (24.1, 30.5), turned to -90 degrees
- moved R22 76.9 mm to (127.9, 56.0), turned to 0 degrees
- moved D8 69.6 mm to (51.4, 38.2)
- moved C24 15.2 mm to (108.2, 49.1)
- moved R18 14.7 mm to (129.3, 46.7), turned to 0 degrees
- moved R27 13.6 mm to (108.2, 47.5)
- moved R19 5.51 mm to (131.1, 48.4), turned to 180 degrees
- moved R21 3.62 mm to (50.3, 49.9)
- moved R17 1.26 mm to (104.6, 37.1), turned to 90 degrees
Connections:
- D8 pad 1: Net-(D10-Pad1) -> Net-(D8-Pad1)
- D8 pad 2: /TIOA0 -> Net-(D8-Pad2)
- FB5 pad 2: Net-(D14-Pad2) -> Net-(D8-Pad2)
- J1 pad A5: unconnected-(J1-PadA5) -> Net-(J1-PadA5)
- J1 pad B5: unconnected-(J1-PadB5) -> Net-(J1-PadB5)
- J6 pad : GND -> (no net)
- R16 pad 1: Net-(D10-Pad1) -> Net-(J1-PadA5)
- R17 pad 1: +3.3V -> /Output/OR Out
- R18 pad 2: +3.3V -> Net-(R18-Pad2)
- R19 pad 2: +3.3V -> Net-(R18-Pad2)
- R21 pad 2: Net-(R21-Pad2) -> /MIDI/MIDI In
- R22 pad 1: Net-(R21-Pad2) -> /Output/EXT In
- R22 pad 2: /MIDI/MIDI In -> GND
- R24 pad 1: Net-(D14-Pad1) -> Net-(D8-Pad1)
- R27 pad 1: Net-(D10-Pad1) -> /Output/OR Out
- U3 pad 1: Net-(R19-Pad1) -> +3.3V
- U3 pad 2: Net-(Q2-Pad3) -> Net-(R19-Pad1)
- U4 pad 3: Net-(Q2-Pad3) -> GND
- U6 pad 2: Net-(D14-Pad1) -> Net-(D8-Pad1)
- U6 pad 3: Net-(D14-Pad2) -> Net-(D8-Pad2)
Routing:
- net /Output/OR Out: track 0.00 -> 68.5 mm, vias 0 -> 3
- net Net-(Q2-Pad3): track 39.8 -> 0.00 mm
- net Net-(D10-Pad1): track 38.3 -> 0.00 mm
- net /Output/EXT In: track 0.00 -> 32.8 mm, vias 0 -> 4
- net Net-(R18-Pad1): track 10.1 -> 26.2 mm
- net /Avg: track 29.4 -> 14.0 mm
- net Net-(D14-Pad2): track 10.2 -> 0.00 mm, vias 1 -> 0
- net Net-(D8-Pad2): track 0.00 -> 10.0 mm, vias 0 -> 1
- net Net-(J1-PadA5): track 0.00 -> 9.27 mm, vias 0 -> 2
- net Net-(U8-Pad12): track 0.00 -> 8.02 mm
- net Net-(R19-Pad1): track 1.99 -> 7.58 mm
- net Net-(U8-Pad11): track 0.00 -> 5.48 mm
- net Net-(D8-Pad1): track 0.00 -> 4.63 mm
- net Net-(D14-Pad1): track 4.63 -> 0.00 mm
- net /TIOA2: track 40.3 -> 44.6 mm
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
Commit message: improved power line filtering
Parts:
- added R29: 10, Resistor_SMD:R_0603_1608Metric_Pad0.98x0.95mm_HandSolder, F.Cu at (33.8, 30.6)
- added REF**: UCSB_IEEE_Logo, Custom_Footprints:UCSB_IEEE_Logo, F.Cu at (28.2, 42.4)
- moved L1 1.53 mm to (33.8, 29.1), turned to 0 degrees
Connections:
- L1 pad 2: +5V -> Net-(L1-Pad2)
Routing:
- net Net-(L1-Pad2): track 0.00 -> 1.62 mm
- net Net-(J1-VBUS-PadA4): track 9.97 -> 8.53 mm
Other:
- rule pad_to_mask_clearance: 0.05 -> 0
- board text added: "Tesla Coil MIDI Interrupter Rev 2 UCSB IEEE Daniel V July 2022"
- board text removed: "Tesla Coil MIDI Interrupter UCSB IEEE Daniel V July 2022"
