File: PCB/Tesla Coil MIDI Synth.kicad_pcb (KiCad board)
At the start: 4 copper layers, 132.1 x 61 mm, 99 parts, among them J1 USB C, J2 JTAG, J3 Expansion, J4 Headphone Output, J5 BNC Output, J6 MIDI Out, J7 MIDI In, SW1 Reset, SW2 Erase, SW3 Rotary Encoder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

Commit message: adjust value to make LCD happy
Parts:
- R29: value 10 -> 3.3
Changed lines of the file:
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@@
         (effects (font (size 1 1) (thickness 0.15)))
     )
-    (fp_text value "10" (at 0 1.43) (layer "F.Fab")
+    (fp_text value "3.3" (at 0 1.43) (layer "F.Fab")
         (effects (font (size 1 1) (thickness 0.15)))
     )
