File: PCB/Tesla Coil MIDI Synth.kicad_sch (KiCad schematic)
At the start: 40 parts, among them J1 USB C, J2 JTAG, J3 Expansion, SW1 Reset, SW2 Erase, SW3 Rotary Encoder, U1 AZ1117-3.3, U2 SAM3A4C, Y1 12MHz

Commit message: fixed PCB
 * Added 5.1k resistors to CC lines on USB-C port
 * Replaced diode OR thing and MOSFET with too low of a threshold voltage with a real OR gate and buffer
 * Fixed polarity of BNC output
 * Made headphone output not murderously loud and asymmetric
 * Added direct in/out to expansion pins
 * Reduced impedance into ADC for average volume level sensing
 * Increased MIDI input pullup resistance
 * Made thermal spokes to copper planes thinner
Parts:
- added R16, R28: 5.1k, Resistor_SMD:R_0603_1608Metric_Pad0.98x0.95mm_HandSolder, symbol Device:R_US
- J3: footprint Connector_PinHeader_2.54mm:PinHeader_2x05_P2.54mm_Vertical -> Connector_PinHeader_2.54mm:PinHeader_2x06_P2.54mm_Vertical; symbol Connector_Generic:Conn_02x05_Odd_Even -> Connector_Generic:Conn_02x06_Odd_Even
Connections:
- net GND: now also R16.2, R28.2
- net at J1.A5 (CC1): now also R16.1
- net at J1.B5 (CC2): now also R28.1
- new net Output/EXT In: J3.11 (Pin_11)
- new net Output/OR Out: J3.12 (Pin_12)
- no-connect marks 42 -> 40
Other:
- sheet Output ports: added EXT In, OR Out; removed none

Commit message: improved power line filtering
Parts:
- added R29: 10, Resistor_SMD:R_0603_1608Metric_Pad0.98x0.95mm_HandSolder, symbol Device:R_US
Connections:
- net +5V: now also R29.2; no longer L1.2
- new net: L1.2, R29.1

Commit message: adjust value to make LCD happy
Parts:
- R29: value 10 -> 3.3
Changed lines of the file:
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@@
       (effects (font (size 1.27 1.27)))
     )
-    (property "Value" "10" (at 55.88 98.3521 90)
+    (property "Value" "3.3" (at 55.88 98.3521 90)
       (effects (font (size 1.27 1.27)))
     )
